File: Freya-sensor.kicad_pcb (KiCad board)
At the start: 2 copper layers, 50 x 15 mm, 24 parts, among them J1 Grove, J2 wires, Q1 BS170, Q2 BS170, U1 BME680, U2 VEML6030, U3 MIC5225-3.3YM5, U4 AS7331

Commit message: Update documentation
Changed lines of the file:
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@@
 		(descr "Bosch BME680 temperature/humidity/pressure/gas sensor")
 		(property "Reference" "U1"
-			(at -2.915 0 180)
+			(at 0 -2.6 180)
 			(layer "F.SilkS")
 			(effects
 				(font
-					(size 1 1)
+					(size 0.8 0.8)
 					(thickness 0.15)
 				)

Commit message: Cleanup PCB & schematic
Parts:
- removed J2: wires, Connector_PinHeader_2.54mm:PinHeader_1x04_P2.54mm_Vertical
Routing:
- net GND: track 41.8 -> 37.5 mm
- net SCL_5v: track 12.8 -> 8.59 mm
- net SDA_5v: track 10.8 -> 6.78 mm
- net +5V: track 26.7 -> 23.9 mm, vias 1 -> 2
Other:
- board text added: "SENSOR Rev. 1.1"
- board text added: "Sensor Rev.: 1.1 by Sanne 'SpuQ' Santens, early 2026"
- board text removed: "SENSOR Rev.: 1.0"
- board text removed: "Sensor Rev.: 1.0 by Sanne 'SpuQ' Santens, late 2024"
