File: Freya-sensor.kicad_sch (KiCad schematic)
At the start: 18 parts, among them J1 Grove, J2 wires, Q1 BS170, Q2 BS170, U1 BME680, U2 VEML6030, U3 MIC5225-3.3YM5, U4 AS7331

Commit message: Update documentation
Other:
- note added: "Address: 0x10"
- note added: "Address: 0x76"
- note removed: "Address: 0x48"
- note removed: "Address: 0x77"
Changed lines of the file:
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@@
 		)
 	)
-	(text "Address: 0x77"
+	(text "Address: 0x76"
 		(exclude_from_sim no)
 		(at 25.4 25.4 0)
@@
 		)
 	)
-	(text "Address: 0x48"
+	(text "Address: 0x10"
 		(exclude_from_sim no)
 		(at 163.83 25.4 0)

Commit message: Cleanup PCB & schematic
Parts:
- removed J2: wires, Connector_PinHeader_2.54mm:PinHeader_1x04_P2.54mm_Vertical, symbol Connector:Conn_01x04_Pin
- J1: value Grove -> JST4.0
Other:
- note added: "Sensor Rev.: 1.1 by Sanne 'SpuQ' Santens, early 2026"
- note removed: "Sensor Rev.: 1.0 by Sanne 'SpuQ' Santens, late 2024"
- moved on the sheet: C1, C2, C3, C4, C5, R5, U1, U2, U3, U4
